File: hw/rev2/sb6502-mk2.kicad_pcb (KiCad board)
At the start: 2 copper layers, 160 x 120 mm, 67 parts, among them J1 Conn_01x03_Pin, J10 Conn_01x04_Socket, J11 Conn_01x04_Socket, J12 Conn_01x08_Socket, J13 Conn_01x08_Socket, J14 Conn_01x08_Socket, J15 Conn_01x08_Socket, J16 Conn_01x08_Socket, J17 Conn_01x04_Socket, J18 Conn_01x04_Socket, J19 Conn_01x02_Socket, J2 Conn_01x03_Pin, J20 Barrel_Jack, J21 Conn_01x02_Socket, J22 Conn_01x06_Socket, J23 Conn_02x02_Counter_Clockwise, J3 DE9_Receptacle, J4 Conn_01x08_Socket, J5 Conn_01x02_Socket, J6 Conn_01x08_Socket, J7 Conn_01x02_Socket, J8 Conn_01x07_Socket, J9 Conn_01x16_Socket, SW1 SW_Push, U1 TC1213, U10 W65C22NxP, U11 74HC138, U2 W65C02SxP, U3 74HC273, U4 ATF22V10, U5 ATF22V10, U6 HM628128, U7 AT28C256, U8 MC68B50, U9 MAX232, X1 1.8432 MHz

Commit message: more work towards PCB-based design
Parts:
- added J24: Conn_01x03_Pin, Connector_PinHeader_2.54mm:PinHeader_1x03_P2.54mm_Vertical, F.Cu at (94.6, 138.0)
- added J25: Conn_01x02_Socket, Connector_PinSocket_2.54mm:PinSocket_1x02_P2.54mm_Vertical, F.Cu at (119.3, 138.0)
- added Q1: 2N7000, Package_TO_SOT_THT:TO-92_Inline, F.Cu at (105.6, 138.2)
- added R8: 3K3, Resistor_THT:R_Axial_DIN0207_L6.3mm_D2.5mm_P7.62mm_Horizontal, F.Cu at (116.2, 137.8)
- added U12: 74HC125, Package_DIP:DIP-14_W7.62mm_Socket, F.Cu at (116.0, 126.8)
- moved J21 56.1 mm to (62.1, 118.2), turned to 0 degrees
- moved C12 17.0 mm to (149.4, 138.6), turned to -90 degrees
- moved SW1 3.45 mm to (125.7, 133.8)
- moved C16 1.59 mm to (134.1, 54.4)
- moved J22 0.40 mm to (48.5, 42.1)
- moved J4 0.30 mm to (30.8, 79.0)
Connections:
- net ~{VP} renamed /Bus Interface/~{VP}
- J9 pad 2: /Bus Interface/A1 -> /Bus Interface/LA1
- J9 pad 3: /Bus Interface/A2 -> /Bus Interface/LA2
- J9 pad 4: /Bus Interface/A3 -> /Bus Interface/LA3
- J9 pad 5: /Bus Interface/A4 -> /Bus Interface/LA4
- U2 pad 10: /Bus Interface/A1 -> /Bus Interface/LA1
- U2 pad 11: /Bus Interface/A2 -> /Bus Interface/LA2
- U2 pad 12: /Bus Interface/A3 -> /Bus Interface/LA3
- U2 pad 13: /Bus Interface/A4 -> /Bus Interface/LA4
- U4 pad 2: /Bus Interface/A2 -> /Bus Interface/LA2
- U4 pad 3: /Bus Interface/A3 -> /Bus Interface/LA3
- U4 pad 4: /Bus Interface/A4 -> /Bus Interface/LA4
Routing:
- net VCC: track 639.3 -> 734.2 mm
- net /Bus Interface/LA2: track 0.00 -> 94.4 mm, vias 0 -> 3
- net /Bus Interface/LA3: track 0.00 -> 90.0 mm, vias 0 -> 3
- net /Bus Interface/LA1: track 0.00 -> 83.8 mm, vias 0 -> 3
- net /Bus Interface/LA4: track 0.00 -> 80.8 mm, vias 0 -> 1
- net /Bus Interface/~{VP}: track 12.9 -> 85.4 mm
- net /Decode/~{IOE1}: track 22.9 -> 77.7 mm, vias 1 -> 2
- net /Decode/~{IOE2}: track 23.6 -> 76.9 mm, vias 1 -> 2
- net /Bus Interface/A1: track 171.2 -> 127.8 mm, vias 5 -> 2
- net Net-(Q1-D): track 0.00 -> 35.5 mm
- net /Bus Interface/A2: track 159.7 -> 130.6 mm, vias 4 -> 2
- net /Bus Interface/A4: track 174.0 -> 145.3 mm, vias 1 -> 0
- net /Bus Interface/A3: track 155.2 -> 135.9 mm, vias 4 -> 2
- net PHI2: track 248.9 -> 261.4 mm
- net ~{RESET}: track 257.7 -> 268.1 mm
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Other:
- board text added: "CTS<"
- board text added: "N.C."
- board text added: "RXD<"
- board text added: "V1"
- board text added: "V2"
- board text added: "VIREO Rev 2"
- board text removed: "<CTS"
- board text removed: "<RXD"
- board text removed: "NC"
- board text removed: "SB6502 Mk2 Rev 2"
- board text removed: "ceharris414@gmail.com"
