File: hw/rev2/bus.kicad_sch (KiCad schematic)
At the start: 10 parts, among them J10 Conn_01x04_Socket, J11 Conn_01x04_Socket, J12 Conn_01x08_Socket, J13 Conn_01x08_Socket, J14 Conn_01x08_Socket, J15 Conn_01x08_Socket, J16 Conn_01x08_Socket, J17 Conn_01x04_Socket, J18 Conn_01x04_Socket, J9 Conn_01x16_Socket

Commit message: more work towards PCB-based design
Connections:
- net A1: no longer J9.2 (Pin_2)
- net A2: no longer J9.3 (Pin_3)
- net A3: no longer J9.4 (Pin_4)
- net A4 renamed LA4
- new net LA1: J9.2 (Pin_2)
- new net LA2: J9.3 (Pin_3)
- new net LA3: J9.4 (Pin_4)

Commit message: hardware revisions
Connections:
- net LA1 is gone; now on net A1: J9.2 (Pin_2)
- net LA2 is gone; now on net A2: J9.3 (Pin_3)
- net LA3 is gone; now on net A3: J9.4 (Pin_4)
- net LA4 renamed A4
Other:
- title: (none) -> Vireo Microcomputer
Changed lines of the file:
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@@
 	(generator_version "9.0")
 	(paper "USLetter")
+	(title_block
+		(title "Vireo Microcomputer")
+		(date "2025-07-27")
+		(rev "2")
+	)
 	(junction
 		(at 158.75 85.09)
@@
 	)
 	(bus_entry
+		(at 45.72 49.53)
+		(size 2.54 2.54)
+		(stroke
+			(width 0)
+			(type default)
+		)
+	)
+	(bus_entry
 		(at 45.72 77.47)
 		(size 2.54 2.54)
@@
 	)
 	(bus_entry
+		(at 45.72 52.07)
+		(size 2.54 2.54)
+		(stroke
+			(width 0)
+			(type default)
+		)
+	)
+	(bus_entry
 		(at 83.82 46.99)
 		(size 2.54 2.54)
@@
 	)
 	(bus_entry
-		(at 33.655 52.07)
-		(size 2.54 2.54)
-		(stroke
-			(width 0)
-			(type default)
-		)
-	)
-	(bus_entry
 		(at 45.72 74.93)
 		(size 2.54 2.54)
@@
 	)
 	(bus_entry
+		(at 45.72 54.61)
+		(size 2.54 2.54)
+		(stroke
+			(width 0)
+			(type default)
+		)
+	)
+	(bus_entry
 		(at 129.54 54.61)
 		(size 2.54 2.54)
@@
 	)
 	(bus_entry
-		(at 33.655 49.53)
-		(size 2.54 2.54)
-		(stroke
-			(width 0)
-			(type default)
-		)
-	)
-	(bus_entry
 		(at 152.4 52.07)
 		(size 2.54 2.54)
@@
 	)
 	(bus_entry
-		(at 33.655 46.99)
+		(at 45.72 46.99)
 		(size 2.54 2.54)
 		(stroke
@@
 	)
 	(bus_entry
-		(at 33.655 54.61)
-		(size 2.54 2.54)
-		(stroke
-			(width 0)
-			(type default)
-		)
-	)
-	(bus_entry
 		(at 64.77 52.07)
 		(size 2.54 2.54)
@@
 	(wire
 		(pts
-			(xy 36.195 49.53) (xy 53.34 49.53)
-		)
-		(stroke
-			(width 0)
-			(type default)
-		)
-	)
-	(wire
-		(pts
 			(xy 151.13 82.55) (xy 161.29 82.55)
 		)
@@
 		)
 	)
-	(bus
-		(pts
-			(xy 30.48 44.45) (xy 33.655 44.45)
-		)
-		(stroke
-			(width 0)
-			(type default)
-		)
-	)
-	(bus
-		(pts
-			(xy 33.655 52.07) (xy 33.655 54.61)
-		)
-		(stroke
-			(width 0)
-			(type default)
-		)
-	)
 	(wire
 		(pts
@@
 	(wire
 		(pts
-			(xy 36.195 57.15) (xy 45.72 57.15)
-		)
-		(stroke
-			(width 0)
-			(type default)
-		)
-	)
-	(wire
-		(pts
 			(xy 154.94 54.61) (xy 160.02 54.61)
 		)
@@
 	(bus
 		(pts
+			(xy 45.72 46.99) (xy 45.72 49.53)
+		)
+		(stroke
+			(width 0)
+			(type default)
+		)
+	)
+	(bus
+		(pts
 			(xy 83.82 46.99) (xy 83.82 49.53)
 		)
@@
 	(bus
 		(pts
-			(xy 45.72 44.45) (xy 45.72 57.15)
+			(xy 45.72 44.45) (xy 45.72 46.99)
 		)
 		(stroke
@@
 		)
 	)
+	(bus
+		(pts
+			(xy 45.72 49.53) (xy 45.72 52.07)
+		)
+		(stroke
+			(width 0)
+			(type default)
+		)
+	)
 	(wire
 		(pts
@@
 		)
 	)
+	(wire
+		(pts
+			(xy 48.26 54.61) (xy 53.34 54.61)
+		)
+		(stroke
+			(width 0)
+			(type default)
+		)
+	)
 	(bus
 		(pts
@@
 		)
 	)
-	(bus
-		(pts
-			(xy 33.655 44.45) (xy 33.655 46.99)
-		)
-		(stroke
-			(width 0)
-			(type default)
-		)
-	)
 	(wire
 		(pts
@@
 		)
 	)
-	(bus
-		(pts
-			(xy 33.655 46.99) (xy 33.655 49.53)
-		)
-		(stroke
-			(width 0)
-			(type default)
-		)
-	)
 	(wire
 		(pts
@@
 		)
 	)
-	(wire
-		(pts
-			(xy 45.72 57.15) (xy 53.34 57.15)
+	(bus
+		(pts
+			(xy 45.72 54.61) (xy 45.72 57.15)
 		)
 		(stroke
@@
 	(wire
 		(pts
-			(xy 36.195 54.61) (xy 53.34 54.61)
+			(xy 48.26 57.15) (xy 53.34 57.15)
 		)
 		(stroke
@@
 		)
 	)
-	(bus
-		(pts
-			(xy 33.655 49.53) (xy 33.655 52.07)
-		)
-		(stroke
-			(width 0)
-			(type default)
-		)
-	)
 	(wire
 		(pts
@@
 		)
 	)
+	(wire
+		(pts
+			(xy 48.26 49.53) (xy 53.34 49.53)
+		)
+		(stroke
+			(width 0)
+			(type default)
+		)
+	)
 	(bus
 		(pts
@@
 		)
 	)
-	(wire
-		(pts
-			(xy 36.195 52.07) (xy 53.34 52.07)
-		)
-		(stroke
-			(width 0)
-			(type default)
-		)
-	)
 	(bus
 		(pts
@@
 	(wire
 		(pts
+			(xy 48.26 52.07) (xy 53.34 52.07)
+		)
+		(stroke
+			(width 0)
+			(type default)
+		)
+	)
+	(wire
+		(pts
 			(xy 132.08 49.53) (xy 137.16 49.53)
 		)
@@
 		(pts
 			(xy 212.09 127) (xy 215.9 127)
+		)
+		(stroke
+			(width 0)
+			(type default)
+		)
+	)
+	(bus
+		(pts
+			(xy 45.72 52.07) (xy 45.72 54.61)
 		)
 		(stroke
@@
 		)
 	)
+	(label "A1"
+		(at 49.53 49.53 0)
+		(effects
+			(font
+				(size 1.27 1.27)
+			)
+			(justify left bottom)
+		)
+	)
 	(label "A0"
 		(at 68.58 46.99 0)
@@
 		)
 	)
-	(label "LA2"
-		(at 36.83 52.07 0)
+	(label "A4"
+		(at 49.53 57.15 0)
 		(effects
 			(font
@@
 		)
 	)
-	(label "LA1"
-		(at 36.83 49.53 0)
-		(effects
-			(font
-				(size 1.27 1.27)
-			)
-			(justify left bottom)
-		)
-	)
 	(label "A7"
 		(at 49.53 64.77 0)
@@
 		)
 	)
+	(label "A3"
+		(at 49.53 54.61 0)
+		(effects
+			(font
+				(size 1.27 1.27)
+			)
+			(justify left bottom)
+		)
+	)
 	(label "A1"
 		(at 68.58 49.53 0)
@@
 		)
 	)
-	(label "LA4"
-		(at 36.83 57.15 0)
-		(effects
-			(font
-				(size 1.27 1.27)
-			)
-			(justify left bottom)
-		)
-	)
 	(label "A9"
 		(at 49.53 69.85 0)
@@
 		)
 	)
-	(label "LA3"
-		(at 36.83 54.61 0)
-		(effects
-			(font
-				(size 1.27 1.27)
-			)
-			(justify left bottom)
-		)
-	)
 	(label "D7"
 		(at 111.76 57.15 0)
@@
 	(label "D2"
 		(at 111.76 44.45 0)
+		(effects
+			(font
+				(size 1.27 1.27)
+			)
+			(justify left bottom)
+		)
+	)
+	(label "A2"
+		(at 49.53 52.07 0)
 		(effects
 			(font
@@
 		)
 	)
-	(hierarchical_label "LA[1..4]"
-		(shape input)
-		(at 30.48 44.45 180)
-		(effects
-			(font
-				(size 1.27 1.27)
-			)
-			(justify right)
-		)
-	)
