File: hw/rev2/cpu.kicad_sch (KiCad schematic)
At the start: 16 parts, among them J24 Conn_01x03_Pin, J25 Conn_01x02_Socket, Q1 2N7000, SW1 SW_Push, U1 TC1213, U12 74HC125, U2 W65C02SxP, X1 1.8432 MHz

Commit message: hardware revisions
Parts:
- J25: value Conn_01x02_Socket -> Conn_01x04_Socket; footprint Connector_PinSocket_2.54mm:PinSocket_1x02_P2.54mm_Vertical -> Connector_PinSocket_2.54mm:PinSocket_1x04_P2.54mm_Vertical; symbol Connector:Conn_01x02_Socket -> Connector:Conn_01x04_Socket
Connections:
- net LA3: now also J25.3 (Pin_3)
- net LA4: now also J25.4 (Pin_4)
Other:
- title: (none) -> Vireo Microcomputer
