File: hw/rev2/io.kicad_sch (KiCad schematic)
At the start: 19 parts, among them J1 Conn_01x03_Pin, J19 Conn_01x02_Socket, J2 Conn_01x03_Pin, J22 Conn_01x06_Socket, J3 DE9_Receptacle, J4 Conn_01x08_Socket, J5 Conn_01x02_Socket, J6 Conn_01x08_Socket, J7 Conn_01x02_Socket, J8 Conn_01x07_Socket, U10 W65C22NxP, U11 74HC138, U8 MC68B50, U9 MAX232

Commit message: hardware revisions
Other:
- title: (none) -> Vireo Microcomputer
Changed lines of the file:
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@@
 	(generator_version "9.0")
 	(paper "USLetter")
+	(title_block
+		(title "Vireo Microcomputer")
+		(date "2025-07-27")
+		(rev "2")
+	)
 	(junction
 		(at 53.34 107.95)
