File: hw/rev2/memory.kicad_sch (KiCad schematic)
At the start: 2 parts, among them U6 HM628128, U7 AT28C256

Commit message: more work towards PCB-based design
Other:
- moved on the sheet: U6, U7

Commit message: hardware revisions
Other:
- title: (none) -> Vireo Microcomputer
Changed lines of the file:
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@@
 	(generator_version "9.0")
 	(paper "USLetter")
+	(title_block
+		(title "Vireo Microcomputer")
+		(date "2025-07-27")
+		(rev "2")
+	)
 	(junction
 		(at 139.7 28.575)
