File: hw/rev2/vireo-rev2.kicad_pcb (KiCad board)
At the start: 2 copper layers, 160 x 120 mm, 72 parts, among them J1 Conn_01x03_Pin, J10 Conn_01x04_Socket, J11 Conn_01x04_Socket, J12 Conn_01x08_Socket, J13 Conn_01x08_Socket, J14 Conn_01x08_Socket, J15 Conn_01x08_Socket, J16 Conn_01x08_Socket, J17 Conn_01x04_Socket, J18 Conn_01x04_Socket, J19 Conn_01x02_Socket, J2 Conn_01x03_Pin, J20 Barrel_Jack, J21 Conn_01x02_Socket, J22 Conn_01x06_Socket, J23 Conn_02x02_Counter_Clockwise, J24 Conn_01x03_Pin, J25 Conn_01x02_Socket, J3 DE9_Receptacle, J4 Conn_01x08_Socket, J5 Conn_01x02_Socket, J6 Conn_01x08_Socket, J7 Conn_01x02_Socket, J8 Conn_01x07_Socket, J9 Conn_01x16_Socket, Q1 2N7000, SW1 SW_Push, U1 TC1213, U10 W65C22NxP, U11 74HC138, U12 74HC125, U2 W65C02SxP, U3 74HC273, U4 ATF22V10, U5 ATF22V10, U6 HM628128, U7 AT28C256, U8 MC68B50, U9 MAX232, X1 1.8432 MHz

Commit message: hardware revisions
Parts:
- added C18: 10µF, Capacitor_THT:CP_Radial_D4.0mm_P2.00mm, F.Cu at (122.4, 37.4)
- C17: value 10µF -> 100nF; footprint Capacitor_THT:CP_Radial_D4.0mm_P2.00mm -> Capacitor_THT:C_Disc_D5.0mm_W2.5mm_P2.50mm
- D2: footprint LED_THT:LED_D5.0mm -> LED_THT:LED_D3.0mm
- J23: value Conn_02x02_Counter_Clockwise -> Conn_02x03_Odd_Even; footprint Connector_PinSocket_2.54mm:PinSocket_2x02_P2.54mm_Vertical -> Connector_PinSocket_2.54mm:PinSocket_2x03_P2.54mm_Vertical
- J25: value Conn_01x02_Socket -> Conn_01x04_Socket; footprint Connector_PinSocket_2.54mm:PinSocket_1x02_P2.54mm_Vertical -> Connector_PinSocket_2.54mm:PinSocket_1x04_P2.54mm_Vertical
- moved C17 101.8 mm to (118.8, 139.2), turned to 0 degrees
- moved J25 11.3 mm to (121.0, 126.8), turned to 0 degrees
- moved C15 8.21 mm to (168.6, 105.0), turned to 0 degrees
- moved D2 3.99 mm to (167.8, 30.2), turned to 180 degrees
- moved J23 1.76 mm to (33.3, 41.0), turned to 90 degrees
- moved SW1 1.46 mm to (127.2, 133.9)
Connections:
- J23 pad 2: VCC -> GND
- J23 pad 3: GND -> VCC
- J25 pad 1: /Bus Interface/LA1 -> /CPU/LA1
- J25 pad 2: /Bus Interface/LA2 -> /CPU/LA2
- J9 pad 2: /Bus Interface/LA1 -> /Bus Interface/A1
- J9 pad 3: /Bus Interface/LA2 -> /Bus Interface/A2
- J9 pad 4: /Bus Interface/LA3 -> /Bus Interface/A3
- J9 pad 5: /Bus Interface/LA4 -> /Bus Interface/A4
- U12 pad 12: /Bus Interface/LA4 -> /CPU/LA4
- U12 pad 2: /Bus Interface/LA1 -> /CPU/LA1
- U12 pad 5: /Bus Interface/LA2 -> /CPU/LA2
- U12 pad 9: /Bus Interface/LA3 -> /CPU/LA3
- U2 pad 10: /Bus Interface/LA1 -> /CPU/LA1
- U2 pad 11: /Bus Interface/LA2 -> /CPU/LA2
- U2 pad 12: /Bus Interface/LA3 -> /CPU/LA3
- U2 pad 13: /Bus Interface/LA4 -> /CPU/LA4
- U4 pad 2: /Bus Interface/LA2 -> /CPU/LA2
- U4 pad 3: /Bus Interface/LA3 -> /CPU/LA3
- U4 pad 4: /Bus Interface/LA4 -> /CPU/LA4
Routing:
- net /Bus Interface/A1: track 127.8 -> 306.6 mm, vias 2 -> 4
- net /Bus Interface/A2: track 130.6 -> 306.6 mm, vias 2 -> 4
- net /Bus Interface/A3: track 135.9 -> 309.3 mm, vias 2 -> 4
- net /Bus Interface/A4: track 145.3 -> 316.0 mm, vias 0 -> 2
- net /Bus Interface/LA2: track 94.4 -> 0.00 mm, vias 3 -> 0
- net /CPU/LA3: track 0.00 -> 93.2 mm, vias 0 -> 4
- net /Bus Interface/LA3: track 90.0 -> 0.00 mm, vias 3 -> 0
- net /CPU/LA2: track 0.00 -> 88.9 mm, vias 0 -> 4
- net /CPU/LA4: track 0.00 -> 84.7 mm, vias 0 -> 2
- net /Bus Interface/LA1: track 83.8 -> 0.00 mm, vias 3 -> 0
- net /Bus Interface/LA4: track 80.8 -> 0.00 mm, vias 1 -> 0
- net /CPU/LA1: track 0.00 -> 69.1 mm, vias 0 -> 2
- net /Decode/~{CONE}: track 147.8 -> 139.9 mm
- net Net-(D2-K): track 7.93 -> 3.80 mm
- net VCC: track 734.2 -> 736.3 mm
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Other:
- board text added: "65C02 @ 1.8432 MHz, 128K RAM, 32K ROM"
- board text added: "LA1"
- board text added: "LA2"
- board text added: "LA3"
- board text added: "LA4"
- board text added: "Rev 2, 2025-07-27"
- board text added: "Vireo"
- board text removed: "V1"
- board text removed: "V2"
- board text removed: "VIREO Rev 2"
